File: KiCad/ControllerConverterForSwitch.kicad_pcb (KiCad board)
At the start: 2 copper layers, 48.3 x 83.4 mm, 12 parts, among them CN1 Conn_01x05, CN2 Conn_01x05, CN3 Conn_01x03, SW1 SW_SPST, SW2 SW_Push, U1 Raspberry Pi Pico, U2 AE-LCNV4-MOSFET

Commit message: add JLCJLCJLCJLC
Other:
- board text added: "JLCJLCJLCJLC"
Changed lines of the file:
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@@
   (gr_line (start 150.495 39.1922) (end 121.285 39.1922) (layer "Edge.Cuts") (width 0.1))
   (gr_line (start 160.02 50.165) (end 156.21 50.165) (layer "Edge.Cuts") (width 0.1))
+  (gr_text "JLCJLCJLCJLC" (at 135.89 119.38) (layer "B.SilkS")
+    (effects (font (size 1 1) (thickness 0.15)) (justify mirror))
+  )
   (gr_text "DET" (at 113.665 83.82) (layer "F.SilkS")
     (effects (font (size 0.8 0.8) (thickness 0.15)))
